File: MagEnc.kicad_pcb (KiCad board)
At the start: 2 copper layers, 24 x 25 mm, 13 parts, among them J101 Conn_01x04_Male, J102 Conn_01x04_Male, J103 Conn_01x04_Male, J104 Conn_01x04_Male, U101 AEAT-8811

Commit message: Update for production
Undate for production
Routing:
- net Net-(J104-Pad4): track 14.1 -> 15.1 mm
- net GND: track 13.9 -> 13.3 mm
- net Net-(J102-Pad3): track 11.4 -> 12.0 mm
- net Net-(J103-Pad3): track 9.57 -> 10.1 mm
Other:
- board text added: "CLK DI DO SEL"
- board text added: "I B A G"
- board text added: "U V W G"
